File: digital_analog_inputs.kicad_sch (KiCad schematic)
At the start: 32 parts

Commit message: Fix minor issues
Other:
- company: (none) -> Dawid Kania
- title: (none) -> PLC IO Module
Changed lines of the file:
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@@
 	(generator_version "8.0")
 	(paper "A4")
+	(title_block
+		(title "PLC IO Module")
+		(rev "1.0.0")
+		(company "Dawid Kania")
+	)
 	(junction
 		(at 259.08 114.3)

Commit message: Generate TME BOM files
Parts:
- C17, C18, C19, C20, C21, C22, C23, C24: Symbol Mouser (none) -> 80-C0805C105Z4VACLR; Symbol TME (none) -> C1206C105K3RAC
- R50, R51, R52, R53, R54, R55, R56, R57: Symbol Mouser (none) -> 71-CRCW080562K0JNEA; Symbol TME (none) -> SMD0805-62K-1%
- R58, R59, R60, R61, R62, R63, R64, R65, R66, R67, R68, R69, R70, R71, R72, R73: Symbol Mouser (none) -> 603-RC0805FR-1010KL; Symbol TME (none) -> RC0805JR-0710K
