File: digital_outputs.kicad_sch (KiCad schematic)
At the start: 64 parts, among them Q1 BCP5516T, Q10 BCP5116TA, Q11 BCP5116TA, Q12 BCP5116TA, Q13 BCP5116TA, Q14 BCP5116TA, Q15 BCP5116TA, Q16 BCP5116TA, Q17 BCP5516T, Q18 BCP5516T, Q19 BCP5516T, Q2 BCP5516T, Q20 BCP5516T, Q21 BCP5516T, Q22 BCP5516T, Q23 BCP5516T, Q24 BCP5516T, Q3 BCP5516T, Q4 BCP5516T, Q5 BCP5516T, Q6 BCP5516T, Q7 BCP5516T, Q8 BCP5516T, Q9 BCP5116TA

Commit message: Fix minor issues
Parts:
- R10, R11, R12, R5, R6, R7, R8, R9: value c -> 500R
- R15, R17, R19, R21, R23, R25, R27, R29: value b -> 5k
- R16, R18, R20, R22, R24, R26, R28, R30: value a -> 100k
- R31, R33, R35, R37, R39, R41, R43, R45: value d -> 500R
- R32, R34, R36, R38, R40, R42, R44, R46: value e -> !00k
Other:
- company: (none) -> Dawid Kania
- title: (none) -> PLC IO Module
Changed lines of the file:
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@@
 	(generator_version "8.0")
 	(paper "A4")
+	(title_block
+		(title "PLC IO Module")
+		(rev "1.0.0")
+		(company "Dawid Kania")
+	)
 	(junction
 		(at 250.19 109.22)
@@
 			)
 		)
-		(property "Value" "a"
+		(property "Value" "100k"
 			(at 110.49 31.7499 0)
 			(effects
@@
 			)
 		)
-		(property "Value" "e"
+		(property "Value" "!00k"
 			(at 110.49 149.8599 0)
 			(effects
@@
 			)
 		)
-		(property "Value" "c"
+		(property "Value" "500R"
 			(at 29.21 48.26 90)
 			(effects
@@
 			)
 		)
-		(property "Value" "b"
+		(property "Value" "5k"
 			(at 110.49 115.5699 0)
 			(effects
@@
 			)
 		)
-		(property "Value" "b"
+		(property "Value" "5k"
 			(at 247.65 115.5699 0)
 			(effects
@@
 			)
 		)
-		(property "Value" "e"
+		(property "Value" "!00k"
 			(at 247.65 76.1999 0)
 			(effects
@@
 			)
 		)
-		(property "Value" "d"
+		(property "Value" "500R"
 			(at 165.1 63.5 90)
 			(effects
@@
 			)
 		)
-		(property "Value" "d"
+		(property "Value" "500R"
 			(at 165.1 137.16 90)
 			(effects
@@
 			)
 		)
-		(property "Value" "a"
+		(property "Value" "100k"
 			(at 176.53 105.4099 0)
 			(effects
@@
 			)
 		)
-		(property "Value" "d"
+		(property "Value" "500R"
 			(at 99.06 63.5 90)
 			(effects
@@
 			)
 		)
-		(property "Value" "e"
+		(property "Value" "!00k"
 			(at 176.53 149.8599 0)
 			(effects
@@
 			)
 		)
-		(property "Value" "c"
+		(property "Value" "500R"
 			(at 236.22 120.65 90)
 			(effects
@@
 			)
 		)
-		(property "Value" "b"
+		(property "Value" "5k"
 			(at 247.65 41.9099 0)
 			(effects
@@
 			)
 		)
-		(property "Value" "a"
+		(property "Value" "100k"
 			(at 247.65 31.7499 0)
 			(effects
@@
 			)
 		)
-		(property "Value" "a"
+		(property "Value" "100k"
 			(at 40.64 33.0199 0)
 			(effects
@@
 			)
 		)
-		(property "Value" "d"
+		(property "Value" "500R"
 			(at 236.22 63.5 90)
 			(effects
@@
 			)
 		)
-		(property "Value" "b"
+		(property "Value" "5k"
 			(at 40.64 116.8399 0)
 			(effects
@@
 			)
 		)
-		(property "Value" "c"
+		(property "Value" "500R"
 			(at 165.1 46.99 90)
 			(effects
@@
 			)
 		)
-		(property "Value" "d"
+		(property "Value" "500R"
 			(at 29.21 64.77 90)
 			(effects
@@
 			)
 		)
-		(property "Value" "e"
+		(property "Value" "!00k"
 			(at 40.64 77.4699 0)
 			(effects
@@
 			)
 		)
-		(property "Value" "c"
+		(property "Value" "500R"
 			(at 165.1 120.65 90)
 			(effects
@@
 			)
 		)
-		(property "Value" "c"
+		(property "Value" "500R"
 			(at 99.06 46.99 90)
 			(effects
@@
 			)
 		)
-		(property "Value" "e"
+		(property "Value" "!00k"
 			(at 247.65 149.8599 0)
 			(effects
@@
 			)
 		)
-		(property "Value" "d"
+		(property "Value" "500R"
 			(at 29.21 138.43 90)
 			(effects
@@
 			)
 		)
-		(property "Value" "b"
+		(property "Value" "5k"
 			(at 110.49 41.9099 0)
 			(effects
@@
 			)
 		)
-		(property "Value" "e"
+		(property "Value" "!00k"
 			(at 176.53 76.1999 0)
 			(effects
@@
 			)
 		)
-		(property "Value" "a"
+		(property "Value" "100k"
 			(at 40.64 106.6799 0)
 			(effects
@@
 			)
 		)
-		(property "Value" "e"
+		(property "Value" "!00k"
 			(at 110.49 76.1999 0)
 			(effects
@@
 			)
 		)
-		(property "Value" "b"
+		(property "Value" "5k"
 			(at 176.53 41.9099 0)
 			(effects
@@
 			)
 		)
-		(property "Value" "a"
+		(property "Value" "100k"
 			(at 176.53 31.7499 0)
 			(effects
@@
 			)
 		)
-		(property "Value" "a"
+		(property "Value" "100k"
 			(at 110.49 105.4099 0)
 			(effects
@@
 			)
 		)
-		(property "Value" "b"
+		(property "Value" "5k"
 			(at 40.64 43.1799 0)
 			(effects
@@
 			)
 		)
-		(property "Value" "c"
+		(property "Value" "500R"
 			(at 29.21 121.92 90)
 			(effects
@@
 			)
 		)
-		(property "Value" "c"
+		(property "Value" "500R"
 			(at 236.22 46.99 90)
 			(effects
@@
 			)
 		)
-		(property "Value" "d"
+		(property "Value" "500R"
 			(at 99.06 137.16 90)
 			(effects
@@
 			)
 		)
-		(property "Value" "b"
+		(property "Value" "5k"
 			(at 176.53 115.5699 0)
 			(effects
@@
 			)
 		)
-		(property "Value" "c"
+		(property "Value" "500R"
 			(at 99.06 120.65 90)
 			(effects
@@
 			)
 		)
-		(property "Value" "a"
+		(property "Value" "100k"
 			(at 247.65 105.4099 0)
 			(effects
@@
 			)
 		)
-		(property "Value" "d"
+		(property "Value" "500R"
 			(at 236.22 137.16 90)
 			(effects
@@
 			)
 		)
-		(property "Value" "e"
+		(property "Value" "!00k"
 			(at 40.64 151.1299 0)
 			(effects

Commit message: Fix minor issues
Parts:
- R32, R34, R36, R38, R40, R42, R44, R46: value !00k -> 100k
Changed lines of the file:
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@@
 			)
 		)
-		(property "Value" "!00k"
+		(property "Value" "100k"
 			(at 110.49 149.8599 0)
 			(effects
@@
 			)
 		)
-		(property "Value" "!00k"
+		(property "Value" "100k"
 			(at 247.65 76.1999 0)
 			(effects
@@
 			)
 		)
-		(property "Value" "!00k"
+		(property "Value" "100k"
 			(at 176.53 149.8599 0)
 			(effects
@@
 			)
 		)
-		(property "Value" "!00k"
+		(property "Value" "100k"
 			(at 40.64 77.4699 0)
 			(effects
@@
 			)
 		)
-		(property "Value" "!00k"
+		(property "Value" "100k"
 			(at 247.65 149.8599 0)
 			(effects
@@
 			)
 		)
-		(property "Value" "!00k"
+		(property "Value" "100k"
 			(at 176.53 76.1999 0)
 			(effects
@@
 			)
 		)
-		(property "Value" "!00k"
+		(property "Value" "100k"
 			(at 110.49 76.1999 0)
 			(effects
@@
 			)
 		)
-		(property "Value" "!00k"
+		(property "Value" "100k"
 			(at 40.64 151.1299 0)
 			(effects

Commit message: Generate TME BOM files
Parts:
- Q1, Q17, Q18, Q19, Q2, Q20, Q21, Q22, Q23, Q24, Q3, Q4, Q5, Q6, Q7, Q8: Symbol Mouser (none) -> 522-BCP5516TA; Symbol TME (none) -> BCP5516TA
- Q10, Q11, Q12, Q13, Q14, Q15, Q16, Q9: Symbol Mouser (none) -> 522-BCP5116TA; Symbol TME (none) -> BCP5116TA
- R10, R11, R12, R31, R33, R35, R37, R39, R41, R43, R45, R5, R6, R7, R8, R9: Symbol Mouser (none) -> 603-RT0805DRE07510RL; Symbol TME (none) -> SMD0805-510R
- R15, R17, R19, R21, R23, R25, R27, R29: Symbol Mouser (none) -> 71-CRCW08055K10JNEA; Symbol TME (none) -> SMD0805-5K1-1%
