File: isolated_connector.kicad_sch (KiCad schematic)
At the start: 6 parts, among them J1 Conn_02x14_Odd_Even, J5 Conn_02x14_Odd_Even, U1 ISO6741

Commit message: Fix minor issues
Other:
- company: (none) -> Dawid Kania
- title: (none) -> PLC IO Module
Changed lines of the file:
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@@
 	(generator_version "8.0")
 	(paper "A4")
+	(title_block
+		(title "PLC IO Module")
+		(rev "1.0.0")
+		(company "Dawid Kania")
+	)
 	(junction
 		(at 227.33 44.45)

Commit message: Generate TME BOM files
Parts:
- C1, C5: Symbol Mouser (none) -> 80-C1206C104K5R7210; Symbol TME (none) -> VJ1206Y104KXBTW1BC
- J1, J5: Symbol Mouser (none) -> -
- JP1: Symbol Mouser (none) -> ====; Symbol TME (none) -> ==
- U1: Symbol Mouser (none) -> 595-ISO6741DWR; Symbol TME (none) -> ---
Changed lines of the file:
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@@
+			)
+		)
+		(property "Symbol Mouser" "-"
+			(at 95.25 59.69 0)
+			(effects
+				(font
+					(size 1.27 1.27)
+				)
+				(hide yes)
+			)
+		)
+		(property "Symbol TME" ""
+			(at 95.25 59.69 0)
+			(effects
+				(font
+					(size 1.27 1.27)
+				)
+				(hide yes)
 			)
 		)
@@
 			)
 		)
+		(property "Symbol Mouser" "80-C1206C104K5R7210"
+			(at 170.18 107.95 0)
+			(effects
+				(font
+					(size 1.27 1.27)
+				)
+				(hide yes)
+			)
+		)
+		(property "Symbol TME" "VJ1206Y104KXBTW1BC"
+			(at 170.18 107.95 0)
+			(effects
+				(font
+					(size 1.27 1.27)
+				)
+				(hide yes)
+			)
+		)
 		(pin "1"
 		)
@@
 		)
 		(property "Description" "3-pole Solder Jumper, pins 1+2 closed/bridged"
+			(at 109.22 144.78 0)
+			(effects
+				(font
+					(size 1.27 1.27)
+				)
+				(hide yes)
+			)
+		)
+		(property "Symbol Mouser" "===="
+			(at 109.22 144.78 0)
+			(effects
+				(font
+					(size 1.27 1.27)
+				)
+				(hide yes)
+			)
+		)
+		(property "Symbol TME" "=="
 			(at 109.22 144.78 0)
 			(effects
@@
 			)
 		)
+		(property "Symbol Mouser" "-"
+			(at 218.44 59.69 0)
+			(effects
+				(font
+					(size 1.27 1.27)
+				)
+				(hide yes)
+			)
+		)
+		(property "Symbol TME" ""
+			(at 218.44 59.69 0)
+			(effects
+				(font
+					(size 1.27 1.27)
+				)
+				(hide yes)
+			)
+		)
 		(pin "13"
 		)
@@
 			)
 		)
+		(property "Symbol Mouser" "595-ISO6741DWR"
+			(at 142.24 130.81 0)
+			(effects
+				(font
+					(size 1.27 1.27)
+				)
+				(hide yes)
+			)
+		)
+		(property "Symbol TME" "---"
+			(at 142.24 130.81 0)
+			(effects
+				(font
+					(size 1.27 1.27)
+				)
+				(hide yes)
+			)
+		)
 		(pin "10"
 		)
@@
 			(at 116.84 107.95 0)
 			(effects
+				(font
+					(size 1.27 1.27)
+				)
+				(hide yes)
+			)
+		)
+		(property "Symbol Mouser" "80-C1206C104K5R7210"
+			(at 116.84 107.95 0)
+			(effects
+				(font
+					(size 1.27 1.27)
+				)
+				(hide yes)
+			)
+		)
+		(property "Symbol TME" "VJ1206Y104KXBTW1BC"
+			(at 116.84 107.95 0)
+			(effects

Commit message: fix problems
Other:
- note added: "TU jest pomyłka MISO i MOSI powinny być zamienione"
Changed lines of the file:
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@@
+		)
+	)
+	(text "TU jest pomyłka\nMISO i MOSI powinny być zamienione\n"
+		(exclude_from_sim no)
+		(at 171.704 144.272 0)
+		(effects
+			(font
+				(size 1.27 1.27)
+			)
 		)
 	)
