File: plc_io_module.kicad_pcb (KiCad board)
At the start: 4 copper layers, 92.5 x 86.4 mm, 145 parts, among them J1 Conn_02x14_Odd_Even, J2 Conn_02x03_Odd_Even, J3 Screw_Terminal_01x02, J4 Screw_Terminal_01x10, J5 Conn_02x14_Odd_Even, Q1 BCP5516T, Q10 BCP5116TA, Q11 BCP5116TA, Q12 BCP5116TA, Q13 BCP5116TA, Q14 BCP5116TA, Q15 BCP5116TA, Q16 BCP5116TA, Q17 BCP5516T, Q18 BCP5516T, Q19 BCP5516T, Q2 BCP5516T, Q20 BCP5516T, Q21 BCP5516T, Q22 BCP5516T, Q23 BCP5516T, Q24 BCP5516T, Q3 BCP5516T, Q4 BCP5516T, Q5 BCP5516T, Q6 BCP5516T, Q7 BCP5516T, Q8 BCP5516T, Q9 BCP5116TA, U1 ISO6741, U2 MC34063AD, U3 STM32F030C6Tx, U4 TLV73333PDBV, Y1 8MHz

Commit message: Fix minor issues
Parts:
- R10, R11, R12, R5, R6, R7, R8, R9: value c -> 500R
- R15, R17, R19, R21, R23, R25, R27, R29: value b -> 5k
- R16, R18, R20, R22, R24, R26, R28, R30: value a -> 100k
- R31, R33, R35, R37, R39, R41, R43, R45: value d -> 500R
- R32, R34, R36, R38, R40, R42, R44, R46: value e -> !00k
- moved C4 1.53 mm to (120.8, 60.5)
Routing:
- net Net-(U2-TC): track 7.58 -> 6.12 mm
Other:
- board text added: "PLC I/O MODULE VERSION 1.0.0 Dawid Kania"
Changed lines of the file:
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@@
 	)
 	(paper "A4")
+	(title_block
+		(title "PLC IO Module")
+		(rev "1.0.0")
+		(company "Dawid Kania")
+	)
 	(layers
 		(0 "F.Cu" signal)
@@
 	(net 128 "Net-(JP4-C)")
 	(net 129 "Net-(U2-Vfb)")
-	(net 130 "Net-(JP601-C)")
+	(net 130 "Net-(JP1-C)")
 	(net 131 "unconnected-(U3-PF7-Pad36)")
 	(net 132 "SIG4_I")
@@
 			(layers "F.Cu" "F.Paste" "F.Mask")
 			(roundrect_rratio 0.25)
-			(net 130 "Net-(JP601-C)")
+			(net 130 "Net-(JP1-C)")
 			(pinfunction "EN1")
 			(pintype "input")
@@
 			)
 		)
-		(property "Value" "a"
+		(property "Value" "100k"
 			(at 0 1.65 90)
 			(layer "F.Fab")
@@
 	(footprint "Capacitor_SMD:C_1206_3216Metric_Pad1.33x1.80mm_HandSolder"
 		(layer "F.Cu")
-		(at 120.65 58.928 180)
+		(at 120.7516 60.452 180)
 		(descr "Capacitor SMD 1206 (3216 Metric), square (rectangular) end terminal, IPC_7351 nominal with elongated pad for handsoldering. (Body size source: IPC-SM-782 page 76, https://www.pcb-3d.com/wordpress/wp-content/uploads/ipc-sm-782a_amendment_1_and_2.pdf), generated with kicad-footprint-generator")
 		(tags "capacitor handsolder")
@@
 			)
 		)
-		(property "Value" "b"
+		(property "Value" "5k"
 			(at 0 1.65 -90)
 			(layer "F.Fab")
@@
 			)
 		)
-		(property "Value" "a"
+		(property "Value" "100k"
 			(at 0 1.65 -90)
 			(layer "F.Fab")
@@
 			)
 		)
-		(property "Value" "c"
+		(property "Value" "500R"
 			(at 0 1.65 90)
 			(layer "F.Fab")
@@
 			)
 		)
-		(property "Value" "c"
+		(property "Value" "500R"
 			(at 0 1.65 90)
 			(layer "F.Fab")
@@
 			)
 		)
-		(property "Value" "d"
+		(property "Value" "500R"
 			(at 0 1.65 -90)
 			(layer "F.Fab")
@@
 			)
 		)
-		(property "Value" "d"
+		(property "Value" "500R"
 			(at 0 1.65 -90)
 			(layer "F.Fab")
@@
 			)
 		)
-		(property "Value" "b"
+		(property "Value" "5k"
 			(at 0 1.65 90)
 			(layer "F.Fab")
@@
 			)
 		)
-		(property "Value" "e"
+		(property "Value" "!00k"
 			(at 0 1.65 -90)
 			(layer "F.Fab")
@@
 			)
 		)
-		(property "Value" "a"
+		(property "Value" "100k"
 			(at 0 1.65 90)
 			(layer "F.Fab")
@@
 			)
 		)
-		(property "Value" "d"
+		(property "Value" "500R"
 			(at 0 1.65 -90)
 			(layer "F.Fab")
@@
 			)
 		)
-		(property "Value" "d"
+		(property "Value" "500R"
 			(at 0 1.65 -90)
 			(layer "F.Fab")
@@
 			)
 		)
-		(property "Value" "e"
+		(property "Value" "!00k"
 			(at 0 1.65 90)
 			(layer "F.Fab")
@@
 			)
 		)
-		(property "Value" "a"
+		(property "Value" "100k"
 			(at 0 1.65 -90)
 			(layer "F.Fab")
@@
 			)
 		)
-		(property "Value" "c"
+		(property "Value" "500R"
 			(at 0 1.65 90)
 			(layer "F.Fab")
@@
 			)
 		)
-		(property "Value" "c"
+		(property "Value" "500R"
 			(at 0 1.65 -90)
 			(layer "F.Fab")
@@
 			)
 		)
-		(property "Value" "b"
+		(property "Value" "5k"
 			(at 0 1.65 -90)
 			(layer "F.Fab")
@@
 			)
 		)
-		(property "Value" "e"
+		(property "Value" "!00k"
 			(at 0 1.65 90)
 			(layer "F.Fab")
@@
 			)
 		)
-		(property "Value" "c"
+		(property "Value" "500R"
 			(at 0 1.65 -90)
 			(layer "F.Fab")
@@
 			)
 		)
-		(property "Value" "d"
+		(property "Value" "500R"
 			(at 0 1.65 -90)
 			(layer "F.Fab")
@@
 			)
 		)
-		(property "Value" "c"
+		(property "Value" "500R"
 			(at 0 1.65 90)
 			(layer "F.Fab")
@@
 			)
 		)
-		(property "Value" "b"
+		(property "Value" "5k"
 			(at 0 1.65 90)
 			(layer "F.Fab")
@@
 			)
 		)
-		(property "Value" "e"
+		(property "Value" "!00k"
 			(at 0 1.65 90)
 			(layer "F.Fab")
@@
 			)
 		)
-		(property "Value" "e"
+		(property "Value" "!00k"
 			(at 0 1.65 90)
 			(layer "F.Fab")
@@
 			)
 		)
-		(property "Value" "d"
+		(property "Value" "500R"
 			(at 0 1.65 -90)
 			(layer "F.Fab")
@@
 			(size 1 1.5)
 			(layers "F.Cu" "F.Mask")
-			(net 130 "Net-(JP601-C)")
+			(net 130 "Net-(JP1-C)")
 			(pinfunction "C")
 			(pintype "passive")
@@
 			)
 		)
-		(property "Value" "a"
+		(property "Value" "100k"
 			(at 0 1.65 90)
 			(layer "F.Fab")
@@
 			)
 		)
-		(property "Value" "c"
+		(property "Value" "500R"
 			(at 0 1.65 -90)
 			(layer "F.Fab")
@@
 			)
 		)
-		(property "Value" "e"
+		(property "Value" "!00k"
 			(at 0 1.65 90)
 			(layer "F.Fab")
@@
 			)
 		)
-		(property "Value" "c"
+		(property "Value" "500R"
 			(at 0 1.65 90)
 			(layer "F.Fab")
@@
 			)
 		)
-		(property "Value" "b"
+		(property "Value" "5k"
 			(at 0 1.65 90)
 			(layer "F.Fab")
@@
 			)
 		)
-		(property "Value" "a"
+		(property "Value" "100k"
 			(at 0 1.65 90)
 			(layer "F.Fab")
@@
 			)
 		)
-		(property "Value" "a"
+		(property "Value" "100k"
 			(at 0 1.65 90)
 			(layer "F.Fab")
@@
 			)
 		)
-		(property "Value" "b"
+		(property "Value" "5k"
 			(at 0 1.65 -90)
 			(layer "F.Fab")
@@
 			)
 		)
-		(property "Value" "e"
+		(property "Value" "!00k"
 			(at 0 1.65 90)
 			(layer "F.Fab")
@@
 			)
 		)
-		(property "Value" "d"
+		(property "Value" "500R"
 			(at 0 1.65 -90)
 			(layer "F.Fab")
@@
 			)
 		)
-		(property "Value" "b"
+		(property "Value" "5k"
 			(at 0 1.65 90)
 			(layer "F.Fab")
@@
 			)
 		)
-		(property "Value" "d"
+		(property "Value" "500R"
 			(at 0 1.65 90)
 			(layer "F.Fab")
@@
 			)
 		)
-		(property "Value" "e"
+		(property "Value" "!00k"
 			(at 0 1.65 90)
 			(layer "F.Fab")
@@
 			)
 		)
-		(property "Value" "b"
+		(property "Value" "5k"
 			(at 0 1.65 90)
 			(layer "F.Fab")
@@
 			)
 		)
-		(property "Value" "a"
+		(property "Value" "100k"
 			(at 0 1.65 90)
 			(layer "F.Fab")
@@
 		)
 	)
+	(gr_text "PLC I/O MODULE\nVERSION 1.0.0\nDawid Kania"
+		(at 159.8676 65.913 0)
+		(layer "F.SilkS")
+		(effects
+			(font
+				(size 1.5 1.5)
+				(thickness 0.3)
+				(bold yes)
+			)
+			(justify left bottom)
+		)
+	)
 	(gr_text "CONFIG_0"
 		(at 117.094 108.712 0)
@@
 		)
 		(height 16.764)
-		(gr_text "78.2320 mm"
+		(gr_text "3080.0000 mils"
 			(at 145.288 149.584 0)
 			(layer "Dwgs.User")
@@
 		)
 		(height -25.908)
-		(gr_text "72.1360 mm"
+		(gr_text "2840.0000 mils"
 			(at 208.512 98.552 90)
 			(layer "Dwgs.User")
@@
 	)
 	(segment
-		(start 119.0875 60.4135)
-		(end 119.126 60.452)
-		(width 0.254)
-		(layer "F.Cu")
-		(net 1)
-	)
-	(segment
 		(start 139.960182 105.192)
 		(end 140.120695 105.031487)
@@
 	)
 	(segment
+		(start 119.1891 61.6843)
+		(end 119.0498 61.8236)
+		(width 0.254)
+		(layer "F.Cu")
+		(net 1)
+	)
+	(segment
 		(start 149.112 122.188)
 		(end 149.86 122.936)
@@
 	)
 	(segment
-		(start 119.0875 58.928)
-		(end 119.0875 60.4135)
+		(start 119.1891 60.452)
+		(end 119.1891 61.6843)
 		(width 0.254)
 		(layer "F.Cu")
@@
 	)
 	(via
-		(at 119.126 60.452)
+		(at 119.0498 61.8236)
 		(size 0.508)
 		(drill 0.254)
@@
 	)
 	(segment
-		(start 122.2125 58.928)
-		(end 122.2125 59.9825)
+		(start 125.033 64.643)
+		(end 123.850003 64.643)
 		(width 0.254)
 		(layer "F.Cu")
@@
 	)
 	(segment
-		(start 125.033 64.643)
-		(end 123.850003 64.643)
+		(start 123.850003 64.643)
+		(end 123.698 64.490997)
 		(width 0.254)
 		(layer "F.Cu")
@@
 	)
 	(segment
-		(start 122.2125 59.9825)
-		(end 122.428 60.198)
+		(start 122.2125 62.1415)
+		(end 122.4534 62.3824)
 		(width 0.254)
 		(layer "F.Cu")
@@
 	)
 	(segment
-		(start 123.850003 64.643)
-		(end 123.698 64.490997)
+		(start 122.3141 60.452)
+		(end 122.2125 60.5536)
+		(width 0.254)
+		(layer "F.Cu")
+		(net 69)
+	)
+	(segment
+		(start 122.2125 60.5536)
+		(end 122.2125 62.1415)
 		(width 0.254)
 		(layer "F.Cu")
@@
 	)
 	(via
-		(at 122.428 60.198)
+		(at 122.4534 62.3824)
 		(size 0.508)
 		(drill 0.254)
@@
 	)
 	(segment
+		(start 123.698 64.490997)
+		(end 122.428 63.220997)
+		(width 0.254)
+		(layer "B.Cu")
+		(net 69)
+	)
+	(segment
 		(start 122.428 63.220997)
-		(end 123.698 64.490997)
+		(end 122.428 62.4078)
 		(width 0.254)
 		(layer "B.Cu")
@@
 	)
 	(segment
-		(start 122.428 60.198)
-		(end 122.428 63.220997)
+		(start 122.428 62.4078)
+		(end 122.4534 62.3824)
 		(width 0.254)
 		(layer "B.Cu")

Commit message: Fix minor issues
Parts:
- R32, R34, R36, R38, R40, R42, R44, R46: value !00k -> 100k
Other:
- board text added: "PLC IO MODULE VERSION 1.0.0 Dawid Kania"
- board text removed: "PLC I/O MODULE VERSION 1.0.0 Dawid Kania"
Changed lines of the file:
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@@
 		(grid_origin 99.06 142.24)
 		(pcbplotparams
-			(layerselection 0x00010fc_ffffffff)
-			(plot_on_all_layers_selection 0x0000000_00000000)
+			(layerselection 0x00311fc_ffffffff)
+			(plot_on_all_layers_selection 0x0001000_00000000)
 			(disableapertmacros no)
-			(usegerberextensions no)
+			(usegerberextensions yes)
 			(usegerberattributes yes)
 			(usegerberadvancedattributes yes)
@@
 			(psa4output no)
 			(plotreference yes)
-			(plotvalue yes)
+			(plotvalue no)
 			(plotfptext yes)
 			(plotinvisibletext no)
 			(sketchpadsonfab no)
-			(subtractmaskfromsilk no)
+			(subtractmaskfromsilk yes)
 			(outputformat 1)
 			(mirror no)
 			(drillshape 0)
 			(scaleselection 1)
-			(outputdirectory "fab_output/board")
+			(outputdirectory "fab_output/gerber")
 		)
 	)
@@
 			)
 		)
-		(property "Value" "!00k"
+		(property "Value" "100k"
 			(at 0 1.65 -90)
 			(layer "F.Fab")
@@
 			)
 		)
-		(property "Value" "!00k"
+		(property "Value" "100k"
 			(at 0 1.65 90)
 			(layer "F.Fab")
@@
 			)
 		)
-		(property "Value" "!00k"
+		(property "Value" "100k"
 			(at 0 1.65 90)
 			(layer "F.Fab")
@@
 			)
 		)
-		(property "Value" "!00k"
+		(property "Value" "100k"
 			(at 0 1.65 90)
 			(layer "F.Fab")
@@
 			)
 		)
-		(property "Value" "!00k"
+		(property "Value" "100k"
 			(at 0 1.65 90)
 			(layer "F.Fab")
@@
 			)
 		)
-		(property "Value" "!00k"
+		(property "Value" "100k"
 			(at 0 1.65 90)
 			(layer "F.Fab")
@@
 			)
 		)
-		(property "Value" "!00k"
+		(property "Value" "100k"
 			(at 0 1.65 90)
 			(layer "F.Fab")
@@
 			)
 		)
-		(property "Value" "!00k"
+		(property "Value" "100k"
 			(at 0 1.65 90)
 			(layer "F.Fab")
@@
 		)
 	)
-	(gr_text "PLC I/O MODULE\nVERSION 1.0.0\nDawid Kania"
+	(gr_text "PLC IO MODULE\nVERSION 1.0.0\nDawid Kania"
 		(at 159.8676 65.913 0)
 		(layer "F.SilkS")

Commit message: Update fabrication files
Other:
- board text removed: "0"
- board text removed: "0 mm"
- board text removed: "0.01 mm"
- board text removed: "0.02"
- board text removed: "0.035 mm"
- board text removed: "0.1 mm"
- board text removed: "0.1270 mm / 0.1270 mm"
- board text removed: "0.1500 mm"
- board text removed: "1"
- board text removed: "1.24 mm"
- board text removed: "1.6000 mm"
- board text removed: "3.3"
- board text removed: "4"
- board text removed: "4.5"
- board text removed: "92.4560 mm x 86.3600 mm"
- board text removed: "B.Cu"
- board text removed: "B.Mask"
- board text removed: "B.Paste"
- board text removed: "B.Silkscreen"
- board text removed: "BOARD CHARACTERISTICS"
- board text removed: "Board Thickness:"
- board text removed: "Board overall dimensions:"
- board text removed: "Bottom Silk Screen"
- board text removed: "Bottom Solder Mask"
- board text removed: "Bottom Solder Paste"
- board text removed: "Castellated pads:"
- board text removed: "Color"
- board text removed: "Copper Finish:"
- board text removed: "Copper Layer Count:"
- board text removed: "Dielectric"
- board text removed: "Edge card connectors:"
- board text removed: "Epsilon R"
- board text removed: "F.Cu"
- board text removed: "F.Mask"
- board text removed: "F.Paste"
- board text removed: "F.Silkscreen"
- board text removed: "FR4"
- board text removed: "FR4 natural"
- board text removed: "Green"
- board text removed: "Impedance Control:"
- board text removed: "In1.Cu"
- board text removed: "In2.Cu"
- board text removed: "Layer Name"
- board text removed: "Loss Tangent"
- board text removed: "Material"
- board text removed: "Min hole diameter:"
- board text removed: "Min track/spacing:"
- board text removed: "No"
- board text removed: "None"
- board text removed: "Not specified"
- board text removed: "Plated Board Edge:"
- board text removed: "Thickness (mm)"
- board text removed: "Top Silk Screen"
- board text removed: "Top Solder Mask"
- board text removed: "Top Solder Paste"
- board text removed: "Type"
- board text removed: "White"
- board text removed: "copper"
- board text removed: "core"
- board text removed: "prepreg"
