File: plc_io_module.kicad_sch (KiCad schematic)
At the start: 24 parts, among them U3 STM32F030C6Tx, Y1 8MHz

Commit message: Fix minor issues
Other:
- company: (none) -> Dawid Kania
- title: (none) -> PLC IO Module
Changed lines of the file:
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@@
 	(generator_version "8.0")
 	(paper "A4")
+	(title_block
+		(title "PLC IO Module")
+		(rev "1.0.0")
+		(company "Dawid Kania")
+	)
 	(junction
 		(at 114.3 54.61)

Commit message: Generate TME BOM files
Parts:
- C12, C16, C2, C3, C6, C7: Symbol Mouser (none) -> 80-C1206C104K5R7210; Symbol TME (none) -> VJ1206Y104KXBTW1BC
- D2: Symbol Mouser (none) -> 604-WP113GDT; Symbol TME (none) -> L-103GDT
- D3: Symbol Mouser (none) -> 604-WP113YDT; Symbol TME (none) -> L-1553YDT
- D4: Symbol Mouser (none) -> 696-SSL-LX2573SRD; Symbol TME (none) -> L-113SURDTK
- H1, H2, H3, H4, JP2, JP3, JP4: Symbol Mouser (none) -> ====; Symbol TME (none) -> ==
- R13, R3: Symbol Mouser (none) -> 603-RC0805FR-1010KL; Symbol TME (none) -> RC0805JR-0710K
- R14: Symbol Mouser (none) -> 71-CRCW080562K0JNEA; Symbol TME (none) -> SMD0805-62K-1%
- R47, R48, R49: Symbol Mouser (none) -> 708-RMCF0805JT300R; Symbol TME (none) -> ERJ6ENF3000V
- U3: Symbol Mouser (none) -> 511-STM32F030C6T6; Symbol TME (none) -> STM32F030C6T6
- Y1: Symbol Mouser (none) -> 73-XT49S800-20; Symbol TME (none) -> 8.00M-HC49-S
