File: power_circuit.kicad_sch (KiCad schematic)
At the start: 16 parts, among them U2 MC34063AD, U4 TLV73333PDBV

Commit message: Fix minor issues
Other:
- company: (none) -> Dawid Kania
- title: (none) -> PLC IO Module
Changed lines of the file:
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@@
 	(generator_version "8.0")
 	(paper "A4")
+	(title_block
+		(title "PLC IO Module")
+		(rev "1.0.0")
+		(company "Dawid Kania")
+	)
 	(junction
 		(at 173.99 78.74)

Commit message: Generate TME BOM files
Parts:
- C10, C14, C15, C9: Symbol Mouser (none) -> 80-C0805C824K4RAUTO; Symbol TME (none) -> 1206B103K101CT
- C11: Symbol Mouser (none) -> 80-EDT477M016S9PAA; Symbol TME (none) -> ZSC00AG4711CARL
- C13: Symbol Mouser (none) -> 140-VZL101M1ETR-0607; Symbol TME (none) -> VS1V101ME077000CE0
- C4: Symbol Mouser (none) -> 791-1206B471K500CT; Symbol TME (none) -> CC1206JRNPOB471
- C8: Symbol Mouser (none) -> 710-865080343009; Symbol TME (none) -> VS1V101ME077000CE0
- D1: Symbol Mouser (none) -> 621-1N5819HW-F; Symbol TME (none) -> 1N5819HWQ-7-F
- L1: Symbol Mouser (none) -> 652-SRR1210-221M; Symbol TME (none) -> DE1205-220
- L2: Symbol Mouser (none) -> 652-SRN6045HA-1R0Y; Symbol TME (none) -> DJNR6045-1R0-S
- R1: Symbol Mouser (none) -> 667-ERA-6AED122V; Symbol TME (none) -> ERA6AEB122V
- R2: Symbol Mouser (none) -> 603-RC0805JR-073K6L; Symbol TME (none) -> ERA6AEB362V
- R4: Symbol Mouser (none) -> 791-RLC32-R330FTP; Symbol TME (none) -> RL1206FR-070R33L
- U2: Symbol Mouser (none) -> 863-MC34063ADG; Symbol TME (none) -> MC34063ADR2G
- U4: Symbol Mouser (none) -> 595-TLV73333PDBVR; Symbol TME (none) -> TLV73333PDBVR
